Commit message: fix: environment hooks & imu_plugin error

File: models/bluerov2_heavy/model.urdf (robot description, URDF)
Before this commit: robot bluerov2_heavy, 10 links, 9 joints
Links:
- link base_link: mass 13.0 -> None
- link dummy_base_link: mass None -> 13.0
- link thruster1: geometry visual mesh filename=package://bluerov2_heavy/meshes/t200_ccw_prop.dae
- link thruster2: geometry visual mesh filename=package://bluerov2_heavy/meshes/t200_ccw_prop.dae
- link thruster3: geometry visual mesh filename=package://bluerov2_heavy/meshes/t200_cw_prop.dae
- link thruster4: geometry visual mesh filename=package://bluerov2_heavy/meshes/t200_cw_prop.dae
- link thruster5: geometry visual mesh filename=package://bluerov2_heavy/meshes/t200_ccw_prop.dae
- link thruster6: geometry visual mesh filename=package://bluerov2_heavy/meshes/t200_cw_prop.dae
- link thruster7: geometry visual mesh filename=package://bluerov2_heavy/meshes/t200_cw_prop.dae
- link thruster8: geometry visual mesh filename=package://bluerov2_heavy/meshes/t200_ccw_prop.dae
Joints:
- joint dummy_joint: child base_link -> dummy_base_link; parent dummy_base_link -> base_link
