Commit message: feat: added front camera
temp

File: models/bluerov2_heavy/model.xacro (robot description, xacro)
@@ -1,4 +1,4 @@
 <?xml version="1.0"?>
-<robot name="bluerov2_heavy">
+<robot name="bluerov2_heavy" xmlns:xacro="http://www.ros.org/wiki/xacro">
   <link name="base_link">
     <visual>
@@ -26,4 +26,11 @@
     <parent link="base_link" />
     <child link="dummy_base_link" />
+  </joint>
+  <link name="front_camera_link">
+  </link>
+  <joint name="front_camera_joint" type="fixed">
+    <parent link="base_link" />
+    <child link="front_camera_link" />
+    <origin xyz="0.093 0.001 0.063" rpy="0 0 0" />
   </joint>
   <gazebo reference="base_link">
@@ -37,5 +44,22 @@
     </sensor>
   </gazebo>
+  <gazebo reference="base_link">
+    <sensor name="front_camera" type="camera">
+      <pose>0.093 0.001 0.063 0 0 0</pose>
+      <always_on>true</always_on>
+      <visualize>true</visualize>
+      <update_rate>30</update_rate>
+      <topic>front_camera/image_raw</topic>
+      <camera name="intel_realsense_r200">
+        <camera_info_topic>camera/camera_info</camera_info_topic>
+      </camera>
+    </sensor>
+  </gazebo>
   <gazebo>
+    <plugin
+      filename="gz-sim-sensors-system"
+      name="gz::sim::systems::Sensors">
+      <render_engine>ogre2</render_engine>
+    </plugin>
     <!-- Hydrodynamics plugin -->
     <plugin
@@ -76,5 +100,5 @@
       <origin rpy="-1.571 0 0" />
       <geometry>
-        <mesh filename="package://bluerov2_heavy/meshes/t200_ccw_prop.dae" />
+        <mesh filename="package://bluerov2_gz/models/bluerov2_heavy/meshes/t200_ccw_prop.dae" />
       </geometry>
     </visual>
@@ -89,5 +113,5 @@
       <origin rpy="-1.571 0 0" />
       <geometry>
-        <mesh filename="package://bluerov2_heavy/meshes/t200_ccw_prop.dae" />
+        <mesh filename="package://bluerov2_gz/models/bluerov2_heavy/meshes/t200_ccw_prop.dae" />
       </geometry>
     </visual>
@@ -102,5 +126,5 @@
       <origin rpy="1.571 0 0" />
       <geometry>
-        <mesh filename="package://bluerov2_heavy/meshes/t200_cw_prop.dae" />
+        <mesh filename="package://bluerov2_gz/models/bluerov2_heavy/meshes/t200_cw_prop.dae" />
       </geometry>
     </visual>
@@ -115,5 +139,5 @@
       <origin rpy="1.571 0 0" />
       <geometry>
-        <mesh filename="package://bluerov2_heavy/meshes/t200_cw_prop.dae" />
+        <mesh filename="package://bluerov2_gz/models/bluerov2_heavy/meshes/t200_cw_prop.dae" />
       </geometry>
     </visual>
@@ -128,5 +152,5 @@
       <origin rpy="-1.571 0 1.571" />
       <geometry>
-        <mesh filename="package://bluerov2_heavy/meshes/t200_ccw_prop.dae" />
+        <mesh filename="package://bluerov2_gz/models/bluerov2_heavy/meshes/t200_ccw_prop.dae" />
       </geometry>
     </visual>
@@ -141,5 +165,5 @@
       <origin rpy="1.571 0 1.571" />
       <geometry>
-        <mesh filename="package://bluerov2_heavy/meshes/t200_cw_prop.dae" />
+        <mesh filename="package://bluerov2_gz/models/bluerov2_heavy/meshes/t200_cw_prop.dae" />
       </geometry>
     </visual>
@@ -154,5 +178,5 @@
       <origin rpy="1.571 0 1.571" />
       <geometry>
-        <mesh filename="package://bluerov2_heavy/meshes/t200_cw_prop.dae" />
+        <mesh filename="package://bluerov2_gz/models/bluerov2_heavy/meshes/t200_cw_prop.dae" />
       </geometry>
     </visual>
@@ -167,5 +191,5 @@
       <origin rpy="-1.571 0 1.571" />
       <geometry>
-        <mesh filename="package://bluerov2_heavy/meshes/t200_ccw_prop.dae" />
+        <mesh filename="package://bluerov2_gz/models/bluerov2_heavy/meshes/t200_ccw_prop.dae" />
       </geometry>
     </visual>

Commit message: feat: add bottom facing camera

File: models/bluerov2_heavy/model.xacro (robot description, xacro)
@@ -59,7 +59,7 @@
     </sensor>
   </gazebo>
-  <gazebo reference="base_link">
+  <gazebo reference="front_camera_link">
     <sensor name="front_camera" type="camera">
-      <pose>0.093 0.001 0.063 0 0 0</pose>
+      <pose>0 0 0 0 0 0</pose>
       <always_on>true</always_on>
       <visualize>true</visualize>
@@ -71,4 +71,43 @@
     </sensor>
   </gazebo>
+  <link name="bottom_camera_link">
+  </link>
+  <!-- Gazebo cameras look along +X; pitching the fixed frame +77 degrees points it down -Z. -->
+  <joint name="bottom_camera_joint" type="fixed">
+    <parent link="base_link" />
+    <child link="bottom_camera_link" />
+    <origin xyz="0.20 0 0.14" rpy="0 1.343903524 0" />
+  </joint>
+  <gazebo reference="bottom_camera_link">
+    <sensor name="bottom_camera" type="camera">
+      <pose>0 0 0 0 0 0</pose>
+      <always_on>true</always_on>
+      <visualize>true</visualize>
+      <update_rate>30</update_rate>
+      <topic>bottom_camera/image_raw</topic>
+      <camera name="bottom_camera">
+        <camera_info_topic>bottom_camera/camera_info</camera_info_topic>
+      </camera>
+    </sensor>
+  </gazebo>
+  <!-- Offset aft of the centered DVL and outside the thruster propeller envelopes. -->
+  <!-- Passive geometry only: this is a future hydrophone attachment frame. -->
+  <link name="hydrophone_link">
+    <visual>
+      <geometry>
+        <cylinder radius="0.015" length="0.04" />
+      </geometry>
+    </visual>
+    <collision>
+      <geometry>
+        <cylinder radius="0.015" length="0.04" />
+      </geometry>
+    </collision>
+  </link>
+  <joint name="hydrophone_joint" type="fixed">
+    <parent link="base_link" />
+    <child link="hydrophone_link" />
+    <origin xyz="-0.20 0 -0.10" rpy="0 0 0" />
+  </joint>
   <gazebo>
     <!-- Water Linked DVL A50, included as its own model rather than copied in,
