Commit message: feat: Water Linked A50 DVL on bluerov2_heavy
Adds models/waterlinked_dvl as a standalone Gazebo model and fixes it to
base_link, publishing gz.msgs.DVLVelocityTracking on /dvl/velocity.

Mount height (dvl_z = -0.10) is measured against the visual mesh, not the
base_link collision box: the DVL ranges visual geometry and the lowest
visual point (battery bracket) is at z = -0.085. The collision slab is a
crude stand-in and sizing off it buries the sensor in the hull.

The sensor needs gz-sim-dvl-system declared at world level; declaring it
inside a model is silently ignored. gz-sim-sensors-system stays here and
must not also be declared in the world, or the render thread crashes with
"Scene already exists with name: scene".

Co-Authored-By: Claude Opus 5 <noreply@anthropic.com>

File: models/bluerov2_heavy/model.xacro (robot description, xacro)
@@ -1,4 +1,19 @@
 <?xml version="1.0"?>
-<robot name="bluerov2_heavy" xmlns:xacro="http://www.ros.org/wiki/xacro">
+<robot name="bluerov2_heavy" xmlns:xacro="http://www.ros.org/wiki/xacro"
+       xmlns:gz="http://gazebosim.org/schema">
+  <!-- DVL mount, relative to base_link.
+       MEASURED, not derived from the collision box: the DVL ranges VISUAL
+       geometry, and the visual mesh's lowest point (battery bracket) is at
+       z = -0.085. Sweeping the sensor down past it, -0.08 still ranges the hull
+       at 0.026 m while -0.09 sees clear. -0.10 leaves ~15 mm of bracket
+       clearance.
+       Do NOT size this off the base_link collision box (0.457x0.575x0.05 at
+       z=0.06) — that slab is a crude stand-in for a ~0.25 m tall vehicle and
+       putting the DVL at -0.02 buries it inside the battery bracket.
+       Echo any change into VISO_POS_Z in banyu_defaults.parm (sign flips: this
+       frame is z-up, ArduPilot's is z-down). -->
+  <xacro:property name="dvl_x" value="0.0" />
+  <xacro:property name="dvl_y" value="0.0" />
+  <xacro:property name="dvl_z" value="-0.10" />
   <link name="base_link">
     <visual>
@@ -57,4 +72,16 @@
   </gazebo>
   <gazebo>
+    <!-- Water Linked DVL A50, included as its own model rather than copied in,
+         then fixed to the hull. Beams point -Z at identity rotation, so a
+         downward mount needs no rotation. -->
+    <include>
+      <uri>model://waterlinked_dvl</uri>
+      <name>dvl</name>
+      <pose>${dvl_x} ${dvl_y} ${dvl_z} 0 0 0</pose>
+    </include>
+    <joint name="dvl_joint" type="fixed">
+      <parent>base_link</parent>
+      <child>dvl::dvl_link</child>
+    </joint>
     <plugin
       filename="gz-sim-sensors-system"
@@ -62,4 +89,10 @@
       <render_engine>ogre2</render_engine>
     </plugin>
+    <!-- The DVL is serviced by gz-sim-dvl-system, which must be declared at
+         WORLD level (see banyu_simulation/worlds/proof_of_readiness.world) —
+         declaring it here is silently ignored. The sensors-system plugin above
+         is still required to create the sensor entity, and must be declared
+         exactly once: having it both here and in the world crashes the render
+         thread with "Scene already exists with name: scene". -->
     <!-- Hydrodynamics plugin -->
     <plugin

Commit message: feat: sonar, hydrophones and Lumen lights on bluerov2_heavy; DVL optional
- down_sonar: Ping2-class echosounder (30 deg gpu_lidar cone, 0.3-100 m)
- banyu::HydrophoneArray plugin: pinger first-arrival times for the survey
- four Lumen spot lights at the mesh's lens centres, aimed along each
  lens normal (10 / 20 deg down), 135 deg beam, emissive lens discs
- the competition vehicle has no DVL: mount now behind xacro arg dvl
  (default false); the DVL model and integration are kept

Co-Authored-By: Claude Opus 5.5 <noreply@anthropic.com>

File: models/bluerov2_heavy/model.xacro (robot description, xacro)
@@ -13,4 +13,8 @@
        Echo any change into VISO_POS_Z in banyu_defaults.parm (sign flips: this
        frame is z-up, ArduPilot's is z-down). -->
+  <!-- The competition vehicle carries no DVL. The mount below and the whole
+       DVL chain (banyu::DvlMavlink, ekf_source_switch, EK3_SRC2 params) are
+       kept for later publishing; pass dvl:=true to put the sensor back. -->
+  <xacro:arg name="dvl" default="false" />
   <xacro:property name="dvl_x" value="0.0" />
   <xacro:property name="dvl_y" value="0.0" />
@@ -71,17 +75,131 @@
     </sensor>
   </gazebo>
+  <!-- Bottom camera, looking straight down (pitch +90 deg turns the camera's
+       +X view axis to -Z). Ahead of the DVL so the DVL stays out of frame. -->
+  <gazebo reference="base_link">
+    <sensor name="bottom_camera" type="camera">
+      <pose>0.15 0 -0.05 0 1.5708 0</pose>
+      <always_on>true</always_on>
+      <visualize>true</visualize>
+      <update_rate>30</update_rate>
+      <topic>bottom_camera/image_raw</topic>
+      <camera name="bottom_camera">
+        <camera_info_topic>bottom_camera/camera_info</camera_info_topic>
+      </camera>
+    </sensor>
+  </gazebo>
+  <!-- Down-facing single-beam echosounder, Blue Robotics Ping2 class: 30 deg
+       beam, 0.3-100 m. Modelled as a 5x5-ray gpu_lidar cone pointing -Z (pitch
+       +90 deg); the altitude reading is the nearest return in the cone, as an
+       echosounder reports first echo. Sits where the DVL mount was, which is
+       already measured clear of the hull (see dvl_z). -->
+  <gazebo reference="base_link">
+    <sensor name="down_sonar" type="gpu_lidar">
+      <pose>0 0 -0.11 0 1.5708 0</pose>
+      <always_on>true</always_on>
+      <visualize>true</visualize>
+      <update_rate>10</update_rate>
+      <topic>down_sonar/scan</topic>
+      <lidar>
+        <scan>
+          <horizontal><samples>5</samples><min_angle>-0.2618</min_angle><max_angle>0.2618</max_angle></horizontal>
+          <vertical><samples>5</samples><min_angle>-0.2618</min_angle><max_angle>0.2618</max_angle></vertical>
+        </scan>
+        <range><min>0.3</min><max>100</max><resolution>0.01</resolution></range>
+        <noise><type>gaussian</type><mean>0</mean><stddev>0.01</stddev></noise>
+      </lidar>
+    </sensor>
+  </gazebo>
+  <!-- Hydrophone array. Gazebo has no acoustics, so banyu_simulation's HydrophoneArray system
+       computes first-arrival times from the true poses. Positions (body frame) must match
+       banyu_detection's pinger_localization `hydrophones` parameter.
+       ponytail: square array under the hull; set to the real mount. -->
+  <gazebo>
+    <plugin filename="BanyuHydrophoneArray" name="banyu::HydrophoneArray">
+      <pinger_model>pinger_green</pinger_model>
+      <acoustic_offset>0 0 -0.186</acoustic_offset>
+      <hydrophone>0.15 0 -0.1</hydrophone>
+      <hydrophone>-0.15 0 -0.1</hydrophone>
+      <hydrophone>0 0.15 -0.1</hydrophone>
+      <hydrophone>0 -0.15 -0.1</hydrophone>
+      <ping_rate>1.0</ping_rate>
+      <jitter>2e-6</jitter>
+      <topic>/banyu/pinger/arrivals</topic>
+    </plugin>
+  </gazebo>
+  <!-- Four Blue Robotics Lumen lights at the lens centres of the four Lumens in
+       bluerov2_heavy.dae (measured off the mesh: lens material "239,239,239",
+       ~36 mm discs). Aimed along each lens's fitted normal: forward, pitched
+       DOWN ~10 deg (top pair) and ~20 deg (bottom pair).
+       Lumen spec: 1500 lm, 135 deg beam in water -> outer_angle 2.356 (full cone).
+       ponytail: diffuse bakes in the water loss over a typical ~1.5 m light
+       path (exp(-attenuation * 1.5), attenuation from main_world's
+       UnderwaterTurbidity) because gz lights only fall off with distance; the
+       overall 1.0 scale is uncalibrated against the scene ambient. Tune
+       lumen_gain against real footage. Backscatter from these lights is not
+       modelled by the turbidity shader, so lit images are optimistic. -->
+  <xacro:property name="lumen_gain" value="1.0" />
+  <xacro:macro name="lumen" params="name x y z pitch">
+    <gazebo reference="base_link">
+      <light name="${name}" type="spot">
+        <pose>${x} ${y} ${z} 0 0 0</pose>
+        <direction>${cos(pitch)} 0 ${-sin(pitch)}</direction>
+        <cast_shadows>false</cast_shadows>
+        <diffuse>${0.41 * lumen_gain} ${0.59 * lumen_gain} ${0.44 * lumen_gain} 1</diffuse>
+        <specular>0.05 0.05 0.05 1</specular>
+        <attenuation>
+          <range>10</range>
+          <constant>0.5</constant>
+          <linear>0</linear>
+          <quadratic>1.0</quadratic>
+        </attenuation>
+        <spot>
+          <inner_angle>1.571</inner_angle>
+          <outer_angle>2.356</outer_angle>
+          <falloff>1.0</falloff>
+        </spot>
+      </light>
+    </gazebo>
+    <!-- Glowing lens so the lamp reads as ON: gz draws no beam, only what it lights. -->
+    <link name="${name}_lens">
+      <visual>
+        <origin xyz="0 0 0" rpy="0 ${pi / 2 + pitch} 0" />
+        <geometry><cylinder radius="0.017" length="0.002" /></geometry>
+      </visual>
+    </link>
+    <joint name="${name}_lens_joint" type="fixed">
+      <parent link="base_link" />
+      <child link="${name}_lens" />
+      <origin xyz="${x + 0.009 * cos(pitch)} ${y} ${z - 0.009 * sin(pitch)}" rpy="0 0 0" />
+    </joint>
+    <gazebo reference="${name}_lens">
+      <visual>
+        <material>
+          <ambient>1 1 1 1</ambient>
+          <diffuse>1 1 1 1</diffuse>
+          <emissive>1 1 0.95 1</emissive>
+        </material>
+      </visual>
+    </gazebo>
+  </xacro:macro>
+  <xacro:lumen name="lumen_top_left" x="0.203" y="0.186" z="0.108" pitch="0.175" />
+  <xacro:lumen name="lumen_top_right" x="0.203" y="-0.186" z="0.108" pitch="0.175" />
+  <xacro:lumen name="lumen_bottom_left" x="0.207" y="0.186" z="-0.057" pitch="0.349" />
+  <xacro:lumen name="lumen_bottom_right" x="0.207" y="-0.186" z="-0.057" pitch="0.349" />
   <gazebo>
     <!-- Water Linked DVL A50, included as its own model rather than copied in,
          then fixed to the hull. Beams point -Z at identity rotation, so a
          downward mount needs no rotation. -->
-    <include>
-      <uri>model://waterlinked_dvl</uri>
-      <name>dvl</name>
-      <pose>${dvl_x} ${dvl_y} ${dvl_z} 0 0 0</pose>
-    </include>
-    <joint name="dvl_joint" type="fixed">
-      <parent>base_link</parent>
-      <child>dvl::dvl_link</child>
-    </joint>
+    <xacro:if value="$(arg dvl)">
+      <include>
+        <uri>model://waterlinked_dvl</uri>
+        <name>dvl</name>
+        <pose>${dvl_x} ${dvl_y} ${dvl_z} 0 0 0</pose>
+      </include>
+      <joint name="dvl_joint" type="fixed">
+        <parent>base_link</parent>
+        <child>dvl::dvl_link</child>
+      </joint>
+    </xacro:if>
     <plugin
       filename="gz-sim-sensors-system"

Commit message: feat: hydrophone frames at lower frame corners, hull shadow blockers
Hydrophone positions live once in the xacro: each becomes a hydrophone_N
TF frame and a HydrophoneArray <hydrophone>. Wide corner baseline keeps
bearing error low with the pinger above or below the vehicle.

Co-Authored-By: Claude Opus 5.5 <noreply@anthropic.com>

File: models/bluerov2_heavy/model.xacro (robot description, xacro)
@@ -111,16 +111,51 @@
     </sensor>
   </gazebo>
-  <!-- Hydrophone array. Gazebo has no acoustics, so banyu_simulation's HydrophoneArray system
-       computes first-arrival times from the true poses. Positions (body frame) must match
-       banyu_detection's pinger_localization `hydrophones` parameter.
-       ponytail: square array under the hull; set to the real mount. -->
+  <!-- Hydrophone array: the positions below are the only copy. Each becomes a
+       hydrophone_N frame (TF via robot_state_publisher, read by pinger_localization)
+       and a <hydrophone> of the HydrophoneArray system, which computes first-arrival
+       times from true poses because Gazebo has no acoustics. N = ADC channel, in order.
+       Mount: the four lower frame corners, inside the side plates and above the skids.
+       Chosen over under-hull / top / front-bracket mounts by bearing error with the hull
+       shadow model below: the pinger is BELOW at the surface transit (a top array would be
+       dry at the 0.15 m float depth) and ABOVE during the survey (the hull shadows an
+       under-hull array); the wide 0.46 x 0.54 m baseline keeps late shadowed picks to a
+       few degrees. ~0.2 m from every thruster, outside both camera views.
+       ponytail: not the real mount (none yet); replace with measured positions. -->
+  <xacro:property name="hydrophone_1_xyz" value="0.23 0.27 -0.09" />   <!-- front left -->
+  <xacro:property name="hydrophone_2_xyz" value="0.23 -0.27 -0.09" />  <!-- front right -->
+  <xacro:property name="hydrophone_3_xyz" value="-0.23 0.27 -0.09" />  <!-- rear left -->
+  <xacro:property name="hydrophone_4_xyz" value="-0.23 -0.27 -0.09" /> <!-- rear right -->
+  <xacro:macro name="hydrophone" params="n xyz">
+    <link name="hydrophone_${n}">
+      <visual>
+        <geometry><cylinder radius="0.01" length="0.03" /></geometry>
+      </visual>
+    </link>
+    <joint name="hydrophone_${n}_joint" type="fixed">
+      <parent link="base_link" />
+      <child link="hydrophone_${n}" />
+      <origin xyz="${xyz}" rpy="0 0 0" />
+    </joint>
+  </xacro:macro>
+  <xacro:hydrophone n="1" xyz="${hydrophone_1_xyz}" />
+  <xacro:hydrophone n="2" xyz="${hydrophone_2_xyz}" />
+  <xacro:hydrophone n="3" xyz="${hydrophone_3_xyz}" />
+  <xacro:hydrophone n="4" xyz="${hydrophone_4_xyz}" />
   <gazebo>
     <plugin filename="BanyuHydrophoneArray" name="banyu::HydrophoneArray">
       <pinger_model>pinger_green</pinger_model>
       <acoustic_offset>0 0 -0.186</acoustic_offset>
-      <hydrophone>0.15 0 -0.1</hydrophone>
-      <hydrophone>-0.15 0 -0.1</hydrophone>
-      <hydrophone>0 0.15 -0.1</hydrophone>
-      <hydrophone>0 -0.15 -0.1</hydrophone>
+      <hydrophone>${hydrophone_1_xyz}</hydrophone>
+      <hydrophone>${hydrophone_2_xyz}</hydrophone>
+      <hydrophone>${hydrophone_3_xyz}</hydrophone>
+      <hydrophone>${hydrophone_4_xyz}</hydrophone>
+      <!-- Hull parts big enough (> ~1 wavelength) to shadow the pinger, body frame
+           min xyz max xyz, measured off bluerov2_heavy.dae. Frame bars, thrusters and the
+           side plates (mostly cut-outs) are left out. -->
+      <blocker>-0.15 -0.057 0.003 0.19 0.057 0.117</blocker>    <!-- electronics tube -->
+      <blocker>-0.14 -0.05 -0.105 0.11 0.05 -0.005</blocker>    <!-- battery tube -->
+      <blocker>-0.21 0.057 0.061 0.21 0.157 0.136</blocker>     <!-- foam, left -->
+      <blocker>-0.21 -0.157 0.061 0.21 -0.057 0.136</blocker>   <!-- foam, right -->
+      <shadow_pick_delay>30e-6</shadow_pick_delay>
       <ping_rate>1.0</ping_rate>
       <jitter>2e-6</jitter>

Commit message: feat: magnetic repair probe under the bow (probe:=false for Core)
Co-Authored-By: Claude Opus 5.5 <noreply@anthropic.com>

File: models/bluerov2_heavy/model.xacro (robot description, xacro)
@@ -163,4 +163,54 @@
     </plugin>
   </gazebo>
+  <!-- Magnetic repair probe (Task 2, handbook 3.3.3): a rigid rod hanging under the bow with
+       a magnet at its tip, held on a light node's switch to "repair" it. The tip is in the
+       bottom camera's view (0.07 m ahead of it, 0.40 m down: ~14 deg off axis), so the
+       mission servos the red ring onto the tip's pixel while it lowers. Matte black so the
+       Lumens do not make it a bright blob in the pipe and light detectors.
+       probe_tip is its own gz link (preserveFixedJoint) so PipelineLights reads the tip pose
+       straight off the model. Mass is about the water it displaces: trim-neutral.
+       ponytail: no real probe yet; replace with the measured mount.
+       Task 2 Core tier needs no probe: probe:=false leaves it off. -->
+  <xacro:arg name="probe" default="true" />
+  <xacro:property name="probe_tip_xyz" value="0.22 0 -0.45" />
+  <xacro:property name="probe_length" value="0.36" />
+  <xacro:if value="$(arg probe)">
+    <link name="probe_tip">
+      <inertial>
+        <origin xyz="0 0 ${probe_length / 2}" />
+        <mass value="0.03" />
+        <inertia ixx="3e-4" iyy="3e-4" izz="1e-6" ixy="0" ixz="0" iyz="0" />
+      </inertial>
+      <visual>
+        <origin xyz="0 0 ${probe_length / 2}" />
+        <geometry><cylinder radius="0.005" length="${probe_length}" /></geometry>
+      </visual>
+      <visual>
+        <origin xyz="0 0 0.01" />
+        <geometry><cylinder radius="0.01" length="0.02" /></geometry>
+      </visual>
+      <collision>
+        <origin xyz="0 0 ${probe_length / 2}" />
+        <geometry><cylinder radius="0.01" length="${probe_length}" /></geometry>
+      </collision>
+    </link>
+    <joint name="probe_tip_joint" type="fixed">
+      <parent link="base_link" />
+      <child link="probe_tip" />
+      <origin xyz="${probe_tip_xyz}" rpy="0 0 0" />
+    </joint>
+    <gazebo reference="probe_tip_joint">
+      <preserveFixedJoint>true</preserveFixedJoint>
+    </gazebo>
+    <gazebo reference="probe_tip">
+      <visual>
+        <material>
+          <ambient>0.02 0.02 0.02 1</ambient>
+          <diffuse>0.02 0.02 0.02 1</diffuse>
+          <specular>0 0 0 1</specular>
+        </material>
+      </visual>
+    </gazebo>
+  </xacro:if>
   <!-- Four Blue Robotics Lumen lights at the lens centres of the four Lumens in
        bluerov2_heavy.dae (measured off the mesh: lens material "239,239,239",
